Commit message: Release Milly SDK 1.0.0 with ROS2 Humble and CI/CD

File: milly_description/urdf/MILLY.urdf (robot description, URDF)
Before this commit: robot MILLY, 9 links, 8 joints
Links:
- link base_link: mass 0.41430094 -> 1.0137217105175504; geometry collision mesh filename=package://milly_description/meshes/J1.stl scale=0.001 0.001 0.001; visual mesh filename=package://milly_description/meshes/J1.stl scale=0.001 0.001 0.001
- link finger_1: mass 0.057499098 -> 0.0387190830608586; geometry collision mesh filename=package://milly_description/meshes/Gripper_Hand_L.stl scale=0.001 0.001 0.001; visual mesh filename=package://milly_description/meshes/Gripper_Hand_L.stl scale=0.001 0.001 0.001
- link finger_2: mass 0.057499098 -> 0.038719083144292205; geometry collision mesh filename=package://milly_description/meshes/Gripper_Hand_R.stl scale=0.001 0.001 0.001; visual mesh filename=package://milly_description/meshes/Gripper_Hand_R.stl scale=0.001 0.001 0.001
- link link_1: mass 1.1339212 -> 1.191749063077993; geometry collision mesh filename=package://milly_description/meshes/J2.stl scale=0.001 0.001 0.001; visual mesh filename=package://milly_description/meshes/J2.stl scale=0.001 0.001 0.001
- link link_2: mass 2.3172244 -> 0.7815897120459003; geometry collision mesh filename=package://milly_description/meshes/J3.stl scale=0.001 0.001 0.001; visual mesh filename=package://milly_description/meshes/J3.stl scale=0.001 0.001 0.001
- link link_3: mass 1.3607867 -> 1.2715523971353635; geometry collision mesh filename=package://milly_description/meshes/J4.stl scale=0.001 0.001 0.001; visual mesh filename=package://milly_description/meshes/J4.stl scale=0.001 0.001 0.001
- link link_4: mass 0.49946308 -> 0.38504353820835835; geometry collision mesh filename=package://milly_description/meshes/J5.stl scale=0.001 0.001 0.001; visual mesh filename=package://milly_description/meshes/J5.stl scale=0.001 0.001 0.001
- link link_5: mass 0.76289173 -> 0.3370698983420428; geometry collision mesh filename=package://milly_description/meshes/J6.stl scale=0.001 0.001 0.001; visual mesh filename=package://milly_description/meshes/J6.stl scale=0.001 0.001 0.001
- link link_6: mass 0.25140424 -> 0.3912467995254684; geometry collision mesh filename=package://milly_description/meshes/J7.stl scale=0.001 0.001 0.001; visual mesh filename=package://milly_description/meshes/J7.stl scale=0.001 0.001 0.001
Joints:
- joint finger_1_joint: axis 0.99584567 0.091057081 0 -> 0.04394457737731645 -0.0009459999999999998 0.9990339948971352; limit lower=-0.02 upper=0.03 effort=20 velocity=0.1 -> lower=0.0 upper=0.05 effort=50.0 velocity=0.1; origin xyz=0.06552811 0.0081136605 -0.11519444 rpy=0 -0 6.0247715e-18 -> xyz=0.05734084000000458 0.004224749999991993 0.10494068000000031 rpy=-1.5707963267948999 -7.630412828596686e-14 1.6149760591513729
- joint finger_2_joint: axis -0.99584567 -0.091057081 0 -> -0.04394457737731632 -0.0009459999999999998 0.9990339948971353; limit lower=-0.02 upper=0.03 effort=20 velocity=0.1 -> lower=0.0 upper=0.05 effort=50.0 velocity=0.1; origin xyz=-0.065921114 -0.0042637112 -0.11519444 rpy=0 -0 6.0247715e-18 -> xyz=-0.055433979999995414 -0.0033001500000080244 0.10505662999999973 rpy=1.5707963267948932 -7.630390836508038e-14 1.6149760591513729
- joint joint_1: axis 0 0 1 -> 0.0 0.0 1.0; limit lower=-2.72 upper=2.72 effort=100 velocity=3.1416 -> lower=-2.8 upper=2.8 effort=50.0 velocity=5.0; origin xyz=0 -0.0375 0.072 rpy=3.1415927 -0 3.3306691e-16 -> xyz=0.0 -0.0575 0.0735 rpy=3.141592653589793 -0.0 0.0
- joint joint_2: axis 0 0 1 -> -3.001013150776784e-23 -0.000857 1.0; limit lower=-0.10 upper=3.24 effort=100 velocity=3.1416 -> lower=-3.2 upper=0.0 effort=50.0 velocity=5.0; origin xyz=0.097892511 3.9308472e-07 -0.066000163 rpy=1.5707963 1.725559e-06 -1.5707963 -> xyz=0.03549999 -3.0419999999997672e-05 -0.06450000000000002 rpy=-3.141592653589793 1.5707963267948966 0
- joint joint_3: axis 0 0 1 -> 3.001013150776784e-23 -0.000857 1.0; limit lower=-0.10 upper=3.07 effort=80 velocity=3.1416 -> lower=-2.75 upper=0.0 effort=50.0 velocity=5.0; origin xyz=-0.2908564 -0.073500339 0.12589251 rpy=-3.1415927 1.5446581e-15 -2.0943934 -> xyz=0.07370373999999999 0.2908022 0.0037491699999999996 rpy=-3.141592653589793 -0.0 0.0
- joint joint_4: axis 0 0 1 -> -0.000857 -0.000782 0.999999; limit lower=-1.85 upper=1.85 effort=50 velocity=3.1416 -> lower=-2.42 upper=2.42 effort=50.0 velocity=5.0; origin xyz=-0.081458652 -0.19444951 0.028 rpy=-1.5707963 -1.5266166 -0.52359878 -> xyz=0.02651155000000003 0.21457556 -0.03181616 rpy=1.5707963267948966 -1.5707963267948966 0
- joint joint_5: axis 0 0 1 -> -0.043843 -0.0008900000000002218 0.999038; limit lower=-1.87 upper=1.92 effort=30 velocity=3.1416 -> lower=-1.84 upper=1.7 effort=50.0 velocity=5.0; origin xyz=-0.0235 1.4210855e-16 -0.0495 rpy=3.1415927 -1.5707963 0 -> xyz=-0.028834410000000005 -0.0012325899999999735 -0.044125700000000004 rpy=-1.5707963267948968 1.0842021724855044e-19 -1.5707963267948966
- joint joint_6: axis 0 0 1 -> -0.0009459999999999999 -0.0012389999999236215 -0.999999; limit lower=-1.60 upper=1.60 effort=20 velocity=3.1416 -> lower=-1.55 upper=1.55 effort=50.0 velocity=5.0; origin xyz=-0.068805556 -0.0019338747 0.023565267 rpy=-1.5707963 1.4354332 -1.5707963 -> xyz=-0.0011629800000000046 0.08397417000000001 0.02895162000000002 rpy=-1.570796326794973 -1.5707963267948963 0
